File: _autosave-Arduino_Basic_Shield.kicad_pcb (KiCad board)
At the start: 2 copper layers, 68.8 x 53.6 mm, 12 parts

Commit message: add autodoc elemente
Parts:
- moved R1 0.25 mm to (139.0, 120.8)
- moved R2 0.25 mm to (135.5, 120.8)
Changed lines of the file:
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@@
 	(footprint "Footprints:RES_0805"
 		(layer "F.Cu")
-		(at 139 121 -90)
+		(at 139 120.75 -90)
 		(property "Reference" "R1"
-			(at -1 -1.5 -90)
+			(at 0.3 -1.8 -90)
 			(unlocked yes)
 			(layer "F.SilkS")
@@
 			)
 		)
-		(property "Footprint" "Footprints:RES_0805"
+		(property "Footprint" "RES_0805"
 			(at 0 0 -90)
 			(unlocked yes)
@@
 		)
 		(fp_text user "${REFERENCE}"
-			(at 0 -3.2 -90)
+			(at 0 -3.2 90)
 			(layer "F.Fab")
 			(effects
@@
 			)
 		)
-		(property "devnote" ""
+		(property "devnote" "LED_3V3"
 			(at 0 0 -90)
 			(unlocked yes)
@@
 			)
 		)
+		(fp_text user "+"
+			(at 1.86 0.295 90)
+			(layer "F.Fab")
+			(effects
+				(font
+					(size 0.48 0.48)
+					(thickness 0.15)
+				)
+			)
+		)
 		(fp_text user "${REFERENCE}"
 			(at -1.9 -9.2 -90)
@@
 				(font
 					(size 1 1)
-					(thickness 0.15)
-				)
-			)
-		)
-		(fp_text user "+"
-			(at 1.86 0.295 90)
-			(layer "F.Fab")
-			(effects
-				(font
-					(size 0.48 0.48)
 					(thickness 0.15)
 				)
@@
 			)
 		)
-		(property "devnote" ""
+		(property "devnote" "LED_5V0"
 			(at 0 0 -90)
 			(unlocked yes)
@@
 			(at 0 -3.85 0)
 			(layer "F.SilkS")
-			(hide yes)
 			(effects
 				(font
@@
 			(at 0 3.85 0)
 			(layer "F.Fab")
-			(hide yes)
 			(effects
 				(font
@@
 	(footprint "Footprints:RES_0805"
 		(layer "F.Cu")
-		(at 135.5 121 -90)
+		(at 135.5 120.75 -90)
 		(property "Reference" "R2"
-			(at -1 -1.5 -90)
+			(at 0.3 -1.8 -90)
 			(unlocked yes)
 			(layer "F.SilkS")
@@
 			)
 		)
-		(property "Footprint" "Footprints:RES_0805"
+		(property "Footprint" "RES_0805"
 			(at 0 0 -90)
 			(unlocked yes)
@@
 		)
 		(property "JLC" "C17513"
-			(at 0 0 -90)
-			(unlocked yes)
-			(layer "F.Fab")
-			(hide yes)
-			(effects
-				(font
-					(size 1 1)
-					(thickness 0.15)
-				)
-			)
-		)
-		(property "devnote" ""
 			(at 0 0 -90)
 			(unlocked yes)
@@
 		)
 		(fp_text user "${REFERENCE}"
-			(at 0 -3.2 -90)
+			(at 0 -3.2 90)
 			(layer "F.Fab")
 			(effects
@@
 			(at 0 -3.85 0)
 			(layer "F.SilkS")
-			(hide yes)
 			(effects
 				(font
@@
 			(at 0 3.85 0)
 			(layer "F.Fab")
-			(hide yes)
 			(effects
 				(font
@@
 			(at 0 -3.85 0)
 			(layer "F.SilkS")
-			(hide yes)
 			(effects
 				(font
@@
 			(at 0 3.85 0)
 			(layer "F.Fab")
-			(hide yes)
 			(effects
 				(font
@@
 			(at 0 -3.85 0)
 			(layer "F.SilkS")
-			(hide yes)
 			(effects
 				(font
@@
 			(at 0 3.85 0)
 			(layer "F.Fab")
-			(hide yes)
 			(effects
 				(font
@@
 		)
 		(fp_text user "${devnote}"
-			(at 2.402679 3.429623 0)
+			(at -3.65 2.75 0)
 			(unlocked yes)
 			(layer "User.9")
@@
 		)
 		(fp_text user "${devnote}"
-			(at -2.564473 3.796932 0)
+			(at -2.45 2.15 180)
 			(unlocked yes)
 			(layer "User.9")
@@
 		)
 		(fp_text user "${devnote}"
-			(at -2.410464 3.796932 0)
+			(at -1.55 2.25 180)
 			(unlocked yes)
 			(layer "User.9")
@@
 		)
 		(fp_text user "${devnote}"
-			(at 2.986055 3.307984 0)
+			(at -1.55 2.25 0)
 			(unlocked yes)
 			(layer "User.9")
