File: untitled.kicad_sch (KiCad schematic)
At the start: 8 parts

Commit message: add autodoc elemente
Parts:
- D1: devnote (none) -> LED_3V3
- D2: devnote (none) -> LED_5V0
- X1: devnote (none) -> Digital 1
- X2: devnote (none) -> Digital 2
- X3: devnote (none) -> Power
- X4: devnote (none) -> Analog
Changed lines of the file:
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@@
+			)
+		)
+		(property "devnote" "Digital 1"
+			(at 82.55 43.18 0)
+			(effects
+				(font
+					(size 1.27 1.27)
+				)
+				(hide yes)
 			)
 		)
@@
 			)
 		)
-		(property "devnote" ""
+		(property "devnote" "LED_5V0"
 			(at 64.262 87.376 0)
 			(show_name yes)
@@
 			)
 		)
-		(property "devnote" ""
-			(at 86.106 78.74 0)
-			(show_name yes)
-			(effects
-				(font
-					(size 1.27 1.27)
-				)
-			)
-		)
 		(pin "2"
 		)
@@
 			)
 		)
-		(property "devnote" ""
+		(property "devnote" "LED_3V3"
 			(at 64.262 78.486 0)
 			(show_name yes)
@@
 			)
 		)
+		(property "devnote" "Power"
+			(at 107.95 43.18 0)
+			(effects
+				(font
+					(size 1.27 1.27)
+				)
+				(hide yes)
+			)
+		)
 		(pin "2"
 		)
@@
 			)
 		)
+		(property "devnote" "Digital 2"
+			(at 95.25 43.18 0)
+			(effects
+				(font
+					(size 1.27 1.27)
+				)
+				(hide yes)
+			)
+		)
 		(pin "4"
 		)
@@
 				(hide yes)
 			)
+		)
+		(property "devnote" "Analog"
+			(at 128.27 43.18 0)
+			(effects
+				(font
+					(size 1.27 1.27)
+				)
+				(hide yes)
+			)
